File: Hardware/E90 Kicad Files/E90.sch (KiCad schematic (older format))
At the start: 93 parts, among them J1 Power Connector Conn_01x02, J10 SDIN Jumper, J11 CS_SDOUT Pre Buffer Test Point, J12 SDOUT Jumper, J13 Audio Connector In Conn_01x03, J14 Conn_02x06_Odd_Even, J15 CS Passthru Jumper Conn_01x02, J16 CS Power Switch Conn_01x02, J17 I2S SDIN Bypass Jumper Conn_0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, J18 PMOD Passthru, J19 I2S SDOUT Bypass Conn_01x02, J2 SWD Connector Conn_02x03, J3 Power Test Point Conn_01x02, J4 BOOT0 Test Point, J6 Audio Connector Out Conn_01x03, J7 MCLK Jumper, J8 WS Jumper, J9 SCLK Jumper, U1 AMS1117-3.3, U5 STM32F407VGT60

Commit message: update untracked
Parts:
- U2, U4: renamed from U?; footprint (none) -> Package_TSSOP_SMD:SOP50P490X110-10N
- U3: renamed from U?; footprint (none) -> Package_SC_70:SOT65P210X110-5N
- U5: footprint LQFP-100_14.0x14.0x0.5P -> Package_QFP:LQFP-100_14x14mm_P0.5mm
Changed lines of the file:
@@
 F 0 "U5" H 5350 9250 50  0000 C CNN
 F 1 "STM32F407VGT60" H 5400 3900 50  0000 C CNN
-F 2 "LQFP-100_14.0x14.0x0.5P" H 3950 4050 50  0001 R CNN
+F 2 "Package_QFP:LQFP-100_14x14mm_P0.5mm" H 3950 4050 50  0001 R CNN
 F 3 "http://www.st.com/st-web-ui/static/active/en/resource/technical/document/datasheet/DM00037051.pdf" H 4650 6650 50  0001 C CNN
 F 4 "C12345" H 4650 6650 50  0001 C CNN "LCSC Part #"
@@
 $EndComp
 $Comp
-L E90_Embedded_DSP:NC7SZ125P5 U?
+L E90_Embedded_DSP:NC7SZ125P5 U3
 U 1 1 5FFD329D
 P 10650 5050
-F 0 "U?" H 10650 5415 50  0000 C CNN
+F 0 "U3" H 10650 5415 50  0000 C CNN
 F 1 "NC7SZ125P5" H 10650 5324 50  0000 C CNN
-F 2 "" H 10550 5250 50  0001 C CNN
+F 2 "Package_SC_70:SOT65P210X110-5N" H 10550 5250 50  0001 C CNN
 F 3 "" H 10550 5250 50  0001 C CNN
 	1    10650 5050
@@
 $EndComp
 $Comp
-L E90_Embedded_DSP:CS4344_CZZ U?
+L E90_Embedded_DSP:CS4344_CZZ U2
 U 1 1 5FFD4C44
 P 12100 2350
-F 0 "U?" H 12400 2900 50  0000 C CNN
+F 0 "U2" H 12400 2900 50  0000 C CNN
 F 1 "CS4344_CZZ" H 12400 2750 50  0000 C CNN
-F 2 "" H 11850 2700 50  0001 C CNN
+F 2 "Package_TSSOP_SMD:SOP50P490X110-10N" H 11850 2700 50  0001 C CNN
 F 3 "" H 11850 2700 50  0001 C CNN
 	1    12100 2350
@@
 $EndComp
 $Comp
-L E90_Embedded_DSP:CS5343_CZZ U?
+L E90_Embedded_DSP:CS5343_CZZ U4
 U 1 1 5FFFCC41
 P 12650 5350
-F 0 "U?" H 13050 5850 50  0000 C CNN
+F 0 "U4" H 13050 5850 50  0000 C CNN
 F 1 "CS5343_CZZ" H 13050 5750 50  0000 C CNN
-F 2 "" H 12200 5550 50  0001 C CNN
+F 2 "Package_TSSOP_SMD:SOP50P490X110-10N" H 12200 5550 50  0001 C CNN
 F 3 "" H 12650 5350 50  0001 C CNN
 	1    12650 5350

Commit message: refactoring PCB
Parts:
- removed J16: CS Power Switch Conn_01x02, Connector_PinHeader_2.54mm:PinHeader_1x02_P2.54mm_Vertical, symbol Connector_Generic:Conn_01x02
Connections:
- net labels removed: CS_POWER
- wire segments 347 -> 350
Changed lines of the file:
@@
 Text GLabel 10550 7300 2    50   Input ~ 0
 CS_SDOUT
-Wire Wire Line
-	11600 7300 11600 7250
 $Comp
 L Connector_Generic:Conn_01x02 J15
@@
 Wire Wire Line
 	10300 7300 10200 7300
-$Comp
-L Connector_Generic:Conn_01x02 J16
-U 1 1 6333A979
-P 12050 7500
-F 0 "J16" V 12100 7100 50  0000 L CNN
-F 1 "CS Power Switch Conn_01x02" V 12200 7100 50  0000 L CNN
-F 2 "Connector_PinHeader_2.54mm:PinHeader_1x02_P2.54mm_Vertical" H 12050 7500 50  0001 C CNN
-F 3 "~" H 12050 7500 50  0001 C CNN
-	1    12050 7500
-	0    1    1    0
-$EndComp
-Wire Wire Line
-	12200 7300 12050 7300
-Text GLabel 12200 7300 2    50   Input ~ 0
-CS_POWER
-Wire Wire Line
-	11950 7300 11600 7300
-$Comp
-L power:+3.3V #PWR032
-U 1 1 61F92C4E
-P 11600 7250
-F 0 "#PWR032" H 11600 7100 50  0001 C CNN
-F 1 "+3.3V" H 11615 7423 50  0000 C CNN
-F 2 "" H 11600 7250 50  0001 C CNN
-F 3 "" H 11600 7250 50  0001 C CNN
-	1    11600 7250
-	1    0    0    -1
-$EndComp
 Wire Notes Line
 	9000 3300 6500 3300
@@
 $EndComp
 Wire Wire Line
-	14750 2150 15000 2150
-Wire Wire Line
-	14300 2250 15000 2250
-Wire Wire Line
 	15000 2350 15000 3050
 Wire Wire Line
 	15000 3050 14650 3050
-Wire Wire Line
-	14750 2150 14750 2500
 Wire Notes Line
 	700  2000 4200 2000
@@
 Wire Wire Line
 	10650 1400 10300 1400
-Text GLabel 10300 1400 0    50   Input ~ 0
-CS_POWER
 Text Notes 6500 3250 0    50   ~ 0
 Switch between onboard (CS) A/D, D/A or external PMOD unit\nJumper Vertical = CS \nJumper horizontal = PMOD
@@
 Wire Wire Line
 	14300 2250 14000 2250
-Connection ~ 14300 2250
 Wire Wire Line
 	14300 2650 14300 2250
@@
 	1    0    0    -1
 $EndComp
-Wire Wire Line
-	15100 5400 15400 5400
 Connection ~ 14700 6000
 Wire Wire Line
@@
 Wire Notes Line
 	16350 3600 16350 6700
-Text GLabel 11500 3950 0    50   Input ~ 0
-CS_POWER
-Wire Wire Line
-	15100 5150 15700 5150
-Wire Wire Line
-	15400 5050 15700 5050
-Wire Wire Line
-	15400 5050 15400 5400
 Wire Wire Line
 	15700 5250 15700 6000
@@
 $EndComp
 Connection ~ 12150 5550
+Wire Wire Line
+	15100 5150 15400 5150
+Wire Wire Line
+	15400 5150 15400 5050
+Wire Wire Line
+	15400 5050 15700 5050
+Wire Wire Line
+	15500 5400 15500 5150
+Wire Wire Line
+	15500 5150 15700 5150
+Wire Wire Line
+	15100 5400 15500 5400
+Wire Wire Line
+	14300 2250 14600 2250
+Wire Wire Line
+	14600 2250 14600 2150
+Wire Wire Line
+	14600 2150 15000 2150
+Connection ~ 14300 2250
+Wire Wire Line
+	14750 2500 14750 2250
+Wire Wire Line
+	14750 2250 15000 2250
+$Comp
+L power:+3.3V #PWR?
+U 1 1 603A73D3
+P 10300 1300
+F 0 "#PWR?" H 10300 1150 50  0001 C CNN
+F 1 "+3.3V" H 10315 1473 50  0000 C CNN
+F 2 "" H 10300 1300 50  0001 C CNN
+F 3 "" H 10300 1300 50  0001 C CNN
+	1    10300 1300
+	1    0    0    -1
+$EndComp
+Wire Wire Line
+	10300 1400 10300 1300
+$Comp
+L power:+3.3V #PWR?
+U 1 1 603C86EB
+P 11500 3850
+F 0 "#PWR?" H 11500 3700 50  0001 C CNN
+F 1 "+3.3V" H 11515 4023 50  0000 C CNN
+F 2 "" H 11500 3850 50  0001 C CNN
+F 3 "" H 11500 3850 50  0001 C CNN
+	1    11500 3850
+	1    0    0    -1
+$EndComp
+Wire Wire Line
+	11500 3950 11500 3850
 $EndSCHEMATC
