File: Hardware/E90 Kicad Files/E90.sch (KiCad schematic (older format))
At the start: 92 parts, among them J1 Power Connector Conn_01x02, J10 SDIN Jumper, J11 CS_SDOUT Pre Buffer Test Point, J12 SDOUT Jumper, J13 Audio Connector In Conn_01x03, J14 Conn_02x06_Odd_Even, J15 CS Passthru Jumper Conn_01x02, J17 I2S SDIN Bypass Jumper Conn_0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, J18 PMOD Passthru, J19 I2S SDOUT Bypass Conn_01x02, J2 SWD Connector Conn_02x03, J3 Power Test Point Conn_01x02, J4 BOOT0 Test Point, J6 Audio Connector Out Conn_01x03, J7 MCLK Jumper, J8 WS Jumper, J9 SCLK Jumper, U1 AMS1117-3.3, U2 CS4344_CZZ, U3 NC7SZ125P5, U4 CS5343_CZZ, U5 STM32F407VGT60

Commit message: added pdf
Parts:
- U3: footprint Package_SC_70:SOT65P210X110-5N -> SC-70-5; LCSC (none) -> C112084
Changed lines of the file:
@@
 F 0 "U3" H 10650 5415 50  0000 C CNN
 F 1 "NC7SZ125P5" H 10650 5324 50  0000 C CNN
-F 2 "Package_SC_70:SOT65P210X110-5N" H 10550 5250 50  0001 C CNN
+F 2 "SC-70-5" H 10550 5250 50  0001 C CNN
 F 3 "" H 10550 5250 50  0001 C CNN
+F 4 "C112084" H 10650 5050 50  0001 C CNN "LCSC"
 	1    10650 5050
 	1    0    0    -1

Commit message: started Pcb rev2
Parts:
- removed J10: SDIN Jumper, Connector_PinHeader_2.54mm:PinHeader_2x02_P2.54mm_Vertical, symbol Connector_Generic:Conn_02x02_Counter_Clockwise
- removed J12: SDOUT Jumper, Connector_PinHeader_2.54mm:PinHeader_2x02_P2.54mm_Vertical, symbol Connector_Generic:Conn_02x02_Counter_Clockwise
- removed J14: Conn_02x06_Odd_Even, Connector_PinHeader_2.54mm:PinHeader_2x06_P2.54mm_Vertical, symbol Connector_Generic:Conn_02x06_Odd_Even
- removed J18: PMOD Passthru, Connector_PinHeader_2.54mm:PinHeader_1x02_P2.54mm_Vertical, symbol Connector_Generic:Conn_01x02
- removed J7: MCLK Jumper, Connector_PinHeader_2.54mm:PinHeader_2x02_P2.54mm_Vertical, symbol Connector_Generic:Conn_02x02_Counter_Clockwise
- removed J8: WS Jumper, Connector_PinHeader_2.54mm:PinHeader_2x02_P2.54mm_Vertical, symbol Connector_Generic:Conn_02x02_Counter_Clockwise
- removed J9: SCLK Jumper, Connector_PinHeader_2.54mm:PinHeader_2x02_P2.54mm_Vertical, symbol Connector_Generic:Conn_02x02_Counter_Clockwise
Connections:
- net labels removed: PMOD_CLK, PMOD_MCLK, PMOD_SDIN, PMOD_SDOUT, PMOD_WS
- wire segments 350 -> 302
- no-connect marks 72 -> 67
Other:
- note removed: "A/D"
- note removed: "Switch between onboard (CS) A/D, D/A or external PMOD unit\nJumper Vertical = CS \nJumper horizontal = PMOD"
- moved on the sheet: C13, C14, C15, C16, C17, C18, C19, C20, C21, C22, FB3, J15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
