File: Hardware/E90 Kicad Files/E90.sch (KiCad schematic (older format))
At the start: 85 parts, among them J1 Power Connector Conn_01x02, J11 CS_SDOUT Pre Buffer Test Point, J13 Audio Connector In Conn_01x03, J15 CS Passthru Jumper Conn_01x02, J17 I2S SDIN Bypass Jumper Conn_0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, J19 I2S SDOUT Bypass Conn_01x02, J2 SWD Connector Conn_02x03, J3 Power Test Point Conn_01x02, J4 BOOT0 Test Point, J6 Audio Connector Out Conn_01x03, U1 AMS1117-3.3, U2 CS4344_CZZ, U3 NC7SZ125P5, U4 CS5343_CZZ, U5 STM32F407VGT60

Commit message: Finished rev2 schem, now onto the PCB
Parts:
- removed C31: 1uF, Capacitor_SMD:C_0603_1608Metric, symbol Device:C_Small
- removed D3: LED_Red, LED_SMD:LED_0603_1608Metric, symbol Device:LED_Small
- removed D4: LED_Green, LED_SMD:LED_0603_1608Metric, symbol Device:LED_Small
- removed D5: LED_Blue, LED_SMD:LED_0603_1608Metric, symbol Device:LED_Small
- removed D6: LED_Yellow, LED_SMD:LED_0603_1608Metric, symbol Device:LED_Small
- removed J1: Power Connector Conn_01x02, Connector_PinHeader_2.54mm:PinHeader_1x02_P2.54mm_Vertical, symbol Connector_Generic:Conn_01x02
- removed J11: CS_SDOUT Pre Buffer Test Point, Connector_PinHeader_2.54mm:PinHeader_1x01_P2.54mm_Vertical, symbol Connector_Generic:Conn_01x01
- removed J13: Audio Connector In Conn_01x03, Connector_PinHeader_2.54mm:PinHeader_1x03_P2.54mm_Vertical, symbol Connector_Generic:Conn_01x03
- removed J15: CS Passthru Jumper Conn_01x02, Connector_PinHeader_2.54mm:PinHeader_1x02_P2.54mm_Vertical, symbol Connector_Generic:Conn_01x02
- removed J17: I2S SDIN Bypass Jumper Conn_01x02, Connector_PinHeader_2.54mm:PinHeader_1x02_P2.54mm_Vertical, symbol Connector_Generic:Conn_01x02
- removed J19: I2S SDOUT Bypass Conn_01x02, Connector_PinHeader_2.54mm:PinHeader_1x02_P2.54mm_Vertical, symbol Connector_Generic:Conn_01x02
- removed J4: BOOT0 Test Point, Connector_PinHeader_2.54mm:PinHeader_1x01_P2.54mm_Vertical, symbol Connector_Generic:Conn_01x01
- removed U3: NC7SZ125P5, SC-70-5, symbol E90_Embedded_DSP:NC7SZ125P5
- added C31: 10uF, Capacitor_SMD:C_0805_2012Metric, symbol Device:CP1_Small
- added C40, C41: 100nF, Capacitor_SMD:C_0402_1005Metric, symbol Device:C_Small
- added D3: B5819W, Diode_SMD:D_SOD-123, symbol Device:D_Schottky_Small
- added D4, D5, D6: LED_RGBA, LED_SMD:19-237-R6GHBHC-A01-2T, symbol Device:LED_RGBA
- added J1, J4: Conn_01x03, Connector_PinHeader_2.54mm:PinHeader_1x03_P2.54mm_Vertical, symbol Connector_Generic:Conn_01x03
- added J10, J9: SJ-63073E, Connector_Audio:CUI_SJ-63073E, symbol Connector:SJ-63073E
- added J5: Conn_01x02, Connector_PinHeader_2.54mm:PinHeader_1x02_P2.54mm_Vertical, symbol Connector_Generic:Conn_01x02
- added J7: USB_B_Mini, Connector_USB:USB_Mini-B_Lumberg_2486_01_Horizontal, symbol Connector:USB_B_Mini
- added J8: Barrel_Jack_Switch, Connector_BarrelJack:BarrelJack_Horizontal, symbol Connector:Barrel_Jack_Switch
- added R21: 10k, Resistor_SMD:R_0603_1608Metric, symbol Device:R_Small_US
- added R22, R23, R24, R25, R26, R27, R28, R29, R30: 1k, Resistor_SMD:R_0603_1608Metric, symbol Device:R_Small_US
- added RV1: 100k, symbol Device:R_POT_TRIM_US
- added RV2: 10k, symbol Device:R_POT_US
- added RV3, RV4, RV5: R_POT_US, symbol Device:R_POT_US
- added U3: TLV2774, Package_DIP:DIP-14_W7.62mm_LongPads, symbol E90_Embedded_DSP:TLV2774
- added U6: USBLC6-2SC6, Package_TO_SOT_SMD:SOT-23-6, symbol Power_Protection:USBLC6-2SC6
- C11: value 2.7nF -> 10uF; LCSC C1609 -> C19702; LCSC Part # C1609 -> C19702; LCSC part number C1609 -> C19702
- C26: value 100nf -> 10uF; footprint Capacitor_SMD:C_0402_1005Metric -> Capacitor_SMD:C_0603_1608Metric; LCSC C1525 -> C19702; LCSC Part # C1525 -> C19702; LCSC part number C1525 -> C19702
- C37: value 180pF -> 100nF; footprint Capacitor_SMD:C_0603_1608Metric -> Capacitor_SMD:C_0402_1005Metric; LCSC C18437 -> C1525; LCSC Part # C18437 -> C1525; LCSC part number C18437 -> C1525
- C6: value 3.3uF -> 10uF; LCSC C51412 -> C19702; LCSC Part # C51412 -> C19702; LCSC part number C51412 -> C19702
- J6: value Audio Connector Out Conn_01x03 -> Conn_01x03
- R12, R9: value 5.1K -> 10k; LCSC C23186 -> C25804; LCSC Part # C23186 -> C25804; LCSC part number C23186 -> C25804
- R15, R16, R17, R18: value 2k2 -> 10k; LCSC C4190 -> C23186; LCSC Part # C4190 -> C23186; LCSC part number C4190 -> C23186
- R19, R20: LCSC C25804 -> C23186; LCSC Part # C25804 -> C23186; LCSC part number C25804 -> C23186
- R3: value 470 -> 10k; LCSC C23179 -> C25804; LCSC Part # C23179 -> C25804; LCSC part number C23179 -> C25804
- R5: value 10K -> 10k
Connections:
- net labels added: +1.65V, +5V, ADC1_IN1, ADC1_IN2, ADC1_IN3, ANALOG_IN, ANALOG_OUT, CS4344_OUT, CS5343_IN, PA0_PWM, PA6_PWM, PA7_PWM, PB0_PWM, PB11_PWM, PB1_PWM, PD12_PWM, PD13_PWM, PD14_PWM, USB_CONN_D+, USB_CONN_D-, USB_D+, USB_D-
- net labels removed: CS_CLK, CS_MCLK, CS_SDIN, CS_SDOUT, CS_WS
- wire segments 302 -> 364
- no-connect marks 67 -> 71
Other:
- note added: "A/D\n"
- note added: "Attenuator Pot\n"
- note added: "Boot mode selection\n"
- note added: "Center Negative Plug"
- note added: "GPIO"
- note added: "I2C"
- note added: "Input Gain Stage"
- note added: "Output Voltage Follower\n"
- note added: "Parameter Pots\n"
- note added: "Quad OP Amp Circuit IN/OUT"
- note added: "RGB LEDs\n"
- note added: "assumes CW 2->1\n\n"
- note removed: "Configure to Boot from Main Flash\n"
- note removed: "Passthru switch connectors\n"
- moved on the sheet: C1, C10, C12, C13, C14, C15, C16, C17, C18, C19, C2, C20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

Commit message: PCB priog
Parts:
- removed C37, C40, C41: 100nF, Capacitor_SMD:C_0402_1005Metric, symbol Device:C_Small
- added H1, H2, H3, H4: MountingHole_Pad, MountingHole:MountingHole_4.3mm_M4_Pad_Via, symbol Mechanical:MountingHole_Pad
- added R31, R32, R33, R34: 10k, Resistor_SMD:R_0603_1608Metric, symbol Device:R_Small_US
- RV1: footprint (none) -> Potentiometer_THT:Potentiometer_Piher_PT-10-V10_Vertical
- RV2, RV3, RV4, RV5: footprint (none) -> Potentiometer_THT:Potentiometer_Bourns_PTV09A-1_Single_Vertical
Connections:
- net +3V3: now also R31.1, R33.1
- net CS4344_OUT: now also RV2.3; no longer RV2.1
- net CS5343_IN: no longer RV1.2
- net GND: now also RV2.1, H1.1, H2.1, H3.1, H4.1, R32.2, R34.2; no longer RV2.3
- net PA6_PWM: now also R22.1; no longer R23.1
- net PA7_PWM: now also R23.1; no longer R22.1
- net PD12_PWM: now also R29.1; no longer R30.1
- net PD13_PWM: now also R30.1; no longer R29.1
- net at U3.1 (1OUT): now also U3.2 (1IN-)
- net at U3.10 (3IN+): now also R33.2, R34.1
- net at U3.3 (1IN+): now also R31.2, R32.1
- net at U3.8 (3OUT): now also U3.9 (3IN-)
- net at D6.2 (GK): now also R30.2; no longer R29.2
- net at D6.3 (BK): now also R29.2; no longer R30.2
- net at D5.1 (RK): now also R26.2; no longer R25.2
- net at D5.2 (GK): now also R25.2; no longer R26.2
- net at R15.1, RV1.3: now also RV1.2
- no-connect marks 71 -> 66
Other:
- note added: "U3A Unused"
- note added: "U3C Unused\n"
- note added: "assumes CW 2->3\n\n"
- note removed: "assumes CW 2->1\n\n"
- moved on the sheet: D6, R25, R26, R29, R30

Commit message: routing
Connections:
- net PB0_PWM: now also R26.1; no longer R27.1
- net PB1_PWM: now also R27.1; no longer R26.1
- net at D4.1 (RK): now also R24.2; no longer R22.2
- net at D4.2 (GK): now also R22.2; no longer R23.2
- net at D4.3 (BK): now also R23.2; no longer R24.2
- no-connect marks 66 -> 65
Other:
- moved on the sheet: R22, R23, R24
Changed lines of the file:
@@
 Text GLabel 7550 9100 0    50   Input ~ 0
 PB11_PWM
+Text GLabel 7550 9300 0    50   Input ~ 0
+PB1_PWM
 Text GLabel 7500 8900 0    50   Input ~ 0
-PB1_PWM
-Text GLabel 7550 9300 0    50   Input ~ 0
 PB0_PWM
+Text GLabel 7600 7950 0    50   Input ~ 0
+PA0_PWM
 Text GLabel 7600 8350 0    50   Input ~ 0
-PA0_PWM
+PA7_PWM
 Text GLabel 7600 8150 0    50   Input ~ 0
-PA7_PWM
-Text GLabel 7600 7950 0    50   Input ~ 0
 PA6_PWM
 Text GLabel 11900 2700 0    50   Input ~ 0
@@
 L Device:R_Small_US R24
 U 1 1 608FE8A5
+P 7750 7950
+F 0 "R24" V 7800 8000 50  0000 C CNN
+F 1 "1k" V 7850 7800 50  0000 C CNN
+F 2 "Resistor_SMD:R_0603_1608Metric" H 7750 7950 50  0001 C CNN
+F 3 "~" H 7750 7950 50  0001 C CNN
+F 4 "C23182" H 7750 7950 50  0001 C CNN "LCSC Part #"
+F 5 "C23182" H 7750 7950 50  0001 C CNN "LCSC part number"
+F 6 "C23182" H 7750 7950 50  0001 C CNN "LCSC"
+	1    7750 7950
+	0    -1   -1   0
+$EndComp
+$Comp
+L Device:R_Small_US R23
+U 1 1 6093AF34
 P 7750 8350
-F 0 "R24" V 7800 8400 50  0000 C CNN
+F 0 "R23" V 7850 8400 50  0000 C CNN
 F 1 "1k" V 7850 8200 50  0000 C CNN
 F 2 "Resistor_SMD:R_0603_1608Metric" H 7750 8350 50  0001 C CNN
@@
 $EndComp
 $Comp
-L Device:R_Small_US R23
-U 1 1 6093AF34
+L Device:R_Small_US R22
+U 1 1 6093B451
 P 7750 8150
-F 0 "R23" V 7850 8200 50  0000 C CNN
+F 0 "R22" V 7850 8200 50  0000 C CNN
 F 1 "1k" V 7850 8000 50  0000 C CNN
 F 2 "Resistor_SMD:R_0603_1608Metric" H 7750 8150 50  0001 C CNN
@@
 	0    -1   -1   0
 $EndComp
-$Comp
-L Device:R_Small_US R22
-U 1 1 6093B451
-P 7750 7950
-F 0 "R22" V 7850 8000 50  0000 C CNN
-F 1 "1k" V 7850 7800 50  0000 C CNN
-F 2 "Resistor_SMD:R_0603_1608Metric" H 7750 7950 50  0001 C CNN
-F 3 "~" H 7750 7950 50  0001 C CNN
-F 4 "C23182" H 7750 7950 50  0001 C CNN "LCSC Part #"
-F 5 "C23182" H 7750 7950 50  0001 C CNN "LCSC part number"
-F 6 "C23182" H 7750 7950 50  0001 C CNN "LCSC"
-	1    7750 7950
-	0    -1   -1   0
-$EndComp
+Wire Wire Line
+	7950 8150 7850 8150
+Wire Wire Line
+	7950 8350 7850 8350
 Wire Wire Line
 	7950 7950 7850 7950
 Wire Wire Line
-	7950 8150 7850 8150
-Wire Wire Line
-	7950 8350 7850 8350
+	7650 7950 7600 7950
 Wire Wire Line
 	7650 8350 7600 8350
 Wire Wire Line
 	7650 8150 7600 8150
-Wire Wire Line
-	7650 7950 7600 7950
 $Comp
 L power:+3.3V #PWR0105
@@
 Connection ~ 13900 7350
 NoConn ~ 6450 2050
-NoConn ~ 2950 10800
 Wire Wire Line
 	7600 10300 7650 10300

Commit message: finished pcb
Parts:
- renumbered RV5 to ADC1_IN1, RV4 to ADC1_IN2, RV3 to ADC1_IN3, RV1 to InputGain1, RV2 to Volume1
Connections:
- net ADC1_IN1: now also ADC1_IN1.2; no longer ADC1_IN3.2
- net ADC1_IN3: now also ADC1_IN3.2; no longer ADC1_IN1.2
- net PB0_PWM: now also R25.1; no longer R26.1
- net PB11_PWM: now also R26.1; no longer R25.1
- net PD12_PWM: now also R28.1; no longer R29.1
- net PD14_PWM: now also R29.1; no longer R28.1
- net at D6.2 (GK): now also R29.2; no longer R30.2
- net at D6.3 (BK): now also R30.2; no longer R29.2
- no-connect marks 65 -> 64
Other:
- moved on the sheet: R29, R30
Changed lines of the file:
@@
 NoConn ~ 5700 7150
 $Comp
-L Device:R_POT_US RV2
+L Device:R_POT_US Volume1
 U 1 1 610194B2
 P 10650 8350
-F 0 "RV2" H 10550 8450 50  0000 R CNN
+F 0 "Volume1" H 10550 8450 50  0000 R CNN
 F 1 "10k" H 10600 8350 50  0000 R CNN
 F 2 "Potentiometer_THT:Potentiometer_Bourns_PTV09A-1_Single_Vertical" H 10650 8350 50  0001 C CNN
@@
 Input Gain Stage
 $Comp
-L Device:R_POT_TRIM_US RV1
+L Device:R_POT_TRIM_US InputGain1
 U 1 1 60AEC4B8
 P 13650 7350
-F 0 "RV1" V 13537 7350 50  0000 C CNN
+F 0 "InputGain1" V 13537 7350 50  0000 C CNN
 F 1 "100k" V 13446 7350 50  0000 C CNN
 F 2 "Potentiometer_THT:Potentiometer_Piher_PT-10-V10_Vertical" H 13650 7350 50  0001 C CNN
@@
 Connection ~ 10750 9850
 $Comp
-L Device:R_POT_US RV3
+L Device:R_POT_US ADC1_IN3
 U 1 1 6083170F
 P 8250 12750
-F 0 "RV3" H 8050 12650 50  0000 R CNN
+F 0 "ADC1_IN3" H 8050 12650 50  0000 R CNN
 F 1 "R_POT_US" H 8150 12750 50  0000 R CNN
 F 2 "Potentiometer_THT:Potentiometer_Bourns_PTV09A-1_Single_Vertical" H 8250 12750 50  0001 C CNN
@@
 	8250 12950 8250 12900
 $Comp
-L Device:R_POT_US RV4
+L Device:R_POT_US ADC1_IN2
 U 1 1 6092E6CE
 P 8250 13700
-F 0 "RV4" H 8350 13000 50  0000 R CNN
+F 0 "ADC1_IN2" H 8350 13000 50  0000 R CNN
 F 1 "R_POT_US" H 8150 13650 50  0000 R CNN
 F 2 "Potentiometer_THT:Potentiometer_Bourns_PTV09A-1_Single_Vertical" H 8250 13700 50  0001 C CNN
@@
 $EndComp
 $Comp
-L Device:R_POT_US RV5
+L Device:R_POT_US ADC1_IN1
 U 1 1 6092EFB7
 P 8250 14650
-F 0 "RV5" H 8000 14550 50  0000 R CNN
+F 0 "ADC1_IN1" H 8000 14550 50  0000 R CNN
 F 1 "R_POT_US" H 8100 14650 50  0000 R CNN
 F 2 "Potentiometer_THT:Potentiometer_Bourns_PTV09A-1_Single_Vertical" H 8250 14650 50  0001 C CNN
@@
 Text GLabel 8000 13700 0    50   Input ~ 0
 ADC1_IN2
+Text GLabel 8000 12750 0    50   Input ~ 0
+ADC1_IN3
+Wire Notes Line
+	7450 12250 9050 12250
+Wire Notes Line
+	9050 12250 9050 15200
+Wire Notes Line
+	9050 15200 7450 15200
+Wire Notes Line
+	7450 15200 7450 12250
 Text GLabel 8050 14650 0    50   Input ~ 0
-ADC1_IN3
-Wire Notes Line
-	7450 12250 9050 12250
-Wire Notes Line
-	9050 12250 9050 15200
-Wire Notes Line
-	9050 15200 7450 15200
-Wire Notes Line
-	7450 15200 7450 12250
-Text GLabel 8000 12750 0    50   Input ~ 0
 ADC1_IN1
 Text Notes 7450 12250 0    50   ~ 0
@@
 Text Notes 6950 7500 0    50   ~ 0
 RGB LEDs\n
+Text GLabel 7600 10100 0    50   Input ~ 0
+PD14_PWM
+Text GLabel 7600 10300 0    50   Input ~ 0
+PD13_PWM
 Text GLabel 7600 9900 0    50   Input ~ 0
-PD14_PWM
-Text GLabel 7600 10100 0    50   Input ~ 0
-PD13_PWM
-Text GLabel 7600 10300 0    50   Input ~ 0
 PD12_PWM
 Wire Wire Line
@@
 Wire Wire Line
 	7950 9300 7850 9300
-Text GLabel 7550 9100 0    50   Input ~ 0
+Text GLabel 7550 8900 0    50   Input ~ 0
 PB11_PWM
 Text GLabel 7550 9300 0    50   Input ~ 0
 PB1_PWM
-Text GLabel 7500 8900 0    50   Input ~ 0
+Text GLabel 7550 9100 0    50   Input ~ 0
 PB0_PWM
 Text GLabel 7600 7950 0    50   Input ~ 0
@@
 NoConn ~ 14650 9550
 NoConn ~ 12500 9550
-NoConn ~ 8650 11200
 NoConn ~ 900  7800
 $Comp
@@
 L Device:R_Small_US R29
 U 1 1 60A9820D
+P 7750 10100
+F 0 "R29" V 7800 10200 50  0000 C CNN
+F 1 "1k" V 7800 10000 50  0000 C CNN
+F 2 "Resistor_SMD:R_0603_1608Metric" H 7750 10100 50  0001 C CNN
+F 3 "~" H 7750 10100 50  0001 C CNN
+F 4 "C23182" H 7750 10100 50  0001 C CNN "LCSC Part #"
+F 5 "C23182" H 7750 10100 50  0001 C CNN "LCSC part number"
+F 6 "C23182" H 7750 10100 50  0001 C CNN "LCSC"
+	1    7750 10100
+	0    -1   -1   0
+$EndComp
+$Comp
+L Device:R_Small_US R30
+U 1 1 60A9872A
 P 7750 10300
-F 0 "R29" V 7800 10400 50  0000 C CNN
+F 0 "R30" V 7800 10400 50  0000 C CNN
 F 1 "1k" V 7800 10200 50  0000 C CNN
 F 2 "Resistor_SMD:R_0603_1608Metric" H 7750 10300 50  0001 C CNN
@@
 F 6 "C23182" H 7750 10300 50  0001 C CNN "LCSC"
 	1    7750 10300
-	0    -1   -1   0
-$EndComp
-$Comp
-L Device:R_Small_US R30
-U 1 1 60A9872A
-P 7750 10100
-F 0 "R30" V 7800 10200 50  0000 C CNN
-F 1 "1k" V 7800 10000 50  0000 C CNN
-F 2 "Resistor_SMD:R_0603_1608Metric" H 7750 10100 50  0001 C CNN
-F 3 "~" H 7750 10100 50  0001 C CNN
-F 4 "C23182" H 7750 10100 50  0001 C CNN "LCSC Part #"
-F 5 "C23182" H 7750 10100 50  0001 C CNN "LCSC part number"
-F 6 "C23182" H 7750 10100 50  0001 C CNN "LCSC"
-	1    7750 10100
 	0    -1   -1   0
 $EndComp
@@
 NoConn ~ 6450 2050
 Wire Wire Line
-	7600 10300 7650 10300
-Wire Wire Line
-	7650 10100 7600 10100
+	7600 10100 7650 10100
+Wire Wire Line
+	7650 10300 7600 10300
 Wire Wire Line
 	8400 10100 8750 10100
@@
 	7850 9900 8000 9900
 Wire Wire Line
+	7850 10300 8000 10300
+Wire Wire Line
 	7850 10100 8000 10100
 Wire Wire Line
-	7850 10300 8000 10300
-Wire Wire Line
-	7650 8900 7500 8900
+	7650 8900 7550 8900
 Wire Wire Line
 	7650 9100 7550 9100

Commit message: added PCB image
Parts:
- C31: LCSC (none) -> C15850
- D4, D5, D6: LCSC (none) -> C60105
- R15, R16, R17, R18, R19, R20, R21, R31, R32, R33, R34: LCSC C23186 -> C25804
- R22, R23, R24, R25, R26, R27, R28, R29, R30: LCSC C23182 -> C21190
- U5: LCSC C12345 -> C919362
- U6: LCSC (none) -> C7519
Changed lines of the file:
@@
 F 4 "C23186" H 14250 8050 50  0001 C CNN "LCSC Part #"
 F 5 "C23186" H 14250 8050 50  0001 C CNN "LCSC part number"
-F 6 "C23186" H 14250 8050 50  0001 C CNN "LCSC"
+F 6 "C25804" H 14250 8050 50  0001 C CNN "LCSC"
 	1    14250 8050
 	0    -1   -1   0
@@
 F 4 "C23186" H 13900 7750 50  0001 C CNN "LCSC Part #"
 F 5 "C23186" H 13900 7750 50  0001 C CNN "LCSC part number"
-F 6 "C23186" H 13900 7750 50  0001 C CNN "LCSC"
+F 6 "C25804" H 13900 7750 50  0001 C CNN "LCSC"
 	1    13900 7750
 	1    0    0    -1
@@
 F 4 "C23186" H 14650 8300 50  0001 C CNN "LCSC Part #"
 F 5 "C23186" H 14650 8300 50  0001 C CNN "LCSC part number"
-F 6 "C23186" H 14650 8300 50  0001 C CNN "LCSC"
+F 6 "C25804" H 14650 8300 50  0001 C CNN "LCSC"
 	1    14650 8300
 	1    0    0    -1
@@
 F 4 "C23186" H 11350 8100 50  0001 C CNN "LCSC Part #"
 F 5 "C23186" H 11350 8100 50  0001 C CNN "LCSC part number"
-F 6 "C23186" H 11350 8100 50  0001 C CNN "LCSC"
+F 6 "C25804" H 11350 8100 50  0001 C CNN "LCSC"
 	1    11350 8100
 	1    0    0    -1
@@
 F 4 "C23186" H 11650 8700 50  0001 C CNN "LCSC Part #"
 F 5 "C23186" H 11650 8700 50  0001 C CNN "LCSC part number"
-F 6 "C23186" H 11650 8700 50  0001 C CNN "LCSC"
+F 6 "C25804" H 11650 8700 50  0001 C CNN "LCSC"
 	1    11650 8700
 	1    0    0    -1
@@
 F 4 "C23186" H 10400 9650 50  0001 C CNN "LCSC Part #"
 F 5 "C23186" H 10400 9650 50  0001 C CNN "LCSC part number"
-F 6 "C23186" H 10400 9650 50  0001 C CNN "LCSC"
+F 6 "C25804" H 10400 9650 50  0001 C CNN "LCSC"
 	1    10400 9650
 	1    0    0    -1
@@
 F 4 "C23186" H 10400 10000 50  0001 C CNN "LCSC Part #"
 F 5 "C23186" H 10400 10000 50  0001 C CNN "LCSC part number"
-F 6 "C23186" H 10400 10000 50  0001 C CNN "LCSC"
+F 6 "C25804" H 10400 10000 50  0001 C CNN "LCSC"
 	1    10400 10000
 	1    0    0    -1
@@
 F 2 "Capacitor_SMD:C_0805_2012Metric" H 10750 10000 50  0001 C CNN
 F 3 "~" H 10750 10000 50  0001 C CNN
+F 4 "C15850" H 10750 10000 50  0001 C CNN "LCSC"
 	1    10750 10000
 	1    0    0    -1
@@
 F 2 "Package_TO_SOT_SMD:SOT-23-6" H 2750 14450 50  0001 C CNN
 F 3 "http://www2.st.com/resource/en/datasheet/CD00050750.pdf" H 3700 14400 50  0001 C CNN
+F 4 "C7519" H 3500 14050 50  0001 C CNN "LCSC"
 	1    3500 14050
 	1    0    0    -1
@@
 F 2 "LED_SMD:19-237-R6GHBHC-A01-2T" H 8150 9050 50  0001 C CNN
 F 3 "~" H 8150 9050 50  0001 C CNN
+F 4 "C60105" H 8150 9100 50  0001 C CNN "LCSC"
 	1    8150 9100
 	1    0    0    -1
@@
 F 2 "LED_SMD:19-237-R6GHBHC-A01-2T" H 8150 8100 50  0001 C CNN
 F 3 "~" H 8150 8100 50  0001 C CNN
+F 4 "C60105" H 8150 8150 50  0001 C CNN "LCSC"
 	1    8150 8150
 	1    0    0    -1
@@
 F 4 "C23182" H 7750 9300 50  0001 C CNN "LCSC Part #"
 F 5 "C23182" H 7750 9300 50  0001 C CNN "LCSC part number"
-F 6 "C23182" H 7750 9300 50  0001 C CNN "LCSC"
+F 6 "C21190" H 7750 9300 50  0001 C CNN "LCSC"
 	1    7750 9300
 	0    -1   -1   0
@@
 F 4 "C23182" H 7750 8900 50  0001 C CNN "LCSC Part #"
 F 5 "C23182" H 7750 8900 50  0001 C CNN "LCSC part number"
-F 6 "C23182" H 7750 8900 50  0001 C CNN "LCSC"
+F 6 "C21190" H 7750 8900 50  0001 C CNN "LCSC"
 	1    7750 8900
 	0    -1   -1   0
@@
 F 4 "C23182" H 7750 9100 50  0001 C CNN "LCSC Part #"
 F 5 "C23182" H 7750 9100 50  0001 C CNN "LCSC part number"
-F 6 "C23182" H 7750 9100 50  0001 C CNN "LCSC"
+F 6 "C21190" H 7750 9100 50  0001 C CNN "LCSC"
 	1    7750 9100
 	0    -1   -1   0
@@
 F 4 "C23182" H 7750 7950 50  0001 C CNN "LCSC Part #"
 F 5 "C23182" H 7750 7950 50  0001 C CNN "LCSC part number"
-F 6 "C23182" H 7750 7950 50  0001 C CNN "LCSC"
+F 6 "C21190" H 7750 7950 50  0001 C CNN "LCSC"
 	1    7750 7950
 	0    -1   -1   0
@@
 F 4 "C23182" H 7750 8350 50  0001 C CNN "LCSC Part #"
 F 5 "C23182" H 7750 8350 50  0001 C CNN "LCSC part number"
-F 6 "C23182" H 7750 8350 50  0001 C CNN "LCSC"
+F 6 "C21190" H 7750 8350 50  0001 C CNN "LCSC"
 	1    7750 8350
 	0    -1   -1   0
@@
 F 4 "C23182" H 7750 8150 50  0001 C CNN "LCSC Part #"
 F 5 "C23182" H 7750 8150 50  0001 C CNN "LCSC part number"
-F 6 "C23182" H 7750 8150 50  0001 C CNN "LCSC"
+F 6 "C21190" H 7750 8150 50  0001 C CNN "LCSC"
 	1    7750 8150
 	0    -1   -1   0
@@
 F 4 "C23182" H 7750 9900 50  0001 C CNN "LCSC Part #"
 F 5 "C23182" H 7750 9900 50  0001 C CNN "LCSC part number"
-F 6 "C23182" H 7750 9900 50  0001 C CNN "LCSC"
+F 6 "C21190" H 7750 9900 50  0001 C CNN "LCSC"
 	1    7750 9900
 	0    -1   -1   0
@@
 F 4 "C23182" H 7750 10100 50  0001 C CNN "LCSC Part #"
 F 5 "C23182" H 7750 10100 50  0001 C CNN "LCSC part number"
-F 6 "C23182" H 7750 10100 50  0001 C CNN "LCSC"
+F 6 "C21190" H 7750 10100 50  0001 C CNN "LCSC"
 	1    7750 10100
 	0    -1   -1   0
@@
 F 4 "C23182" H 7750 10300 50  0001 C CNN "LCSC Part #"
 F 5 "C23182" H 7750 10300 50  0001 C CNN "LCSC part number"
-F 6 "C23182" H 7750 10300 50  0001 C CNN "LCSC"
+F 6 "C21190" H 7750 10300 50  0001 C CNN "LCSC"
 	1    7750 10300
 	0    -1   -1   0
@@
 F 4 "C12345" H 4800 9150 50  0001 C CNN "LCSC Part #"
 F 5 "C12345" H 4800 9150 50  0001 C CNN "LCSC part number"
-F 6 "C12345" H 4800 9150 50  0001 C CNN "LCSC"
+F 6 "C919362" H 4800 9150 50  0001 C CNN "LCSC"
 	1    4800 9150
 	1    0    0    -1
@@
 F 2 "LED_SMD:19-237-R6GHBHC-A01-2T" H 8200 10050 50  0001 C CNN
 F 3 "~" H 8200 10050 50  0001 C CNN
+F 4 "C60105" H 8200 10100 50  0001 C CNN "LCSC"
 	1    8200 10100
 	1    0    0    -1
@@
 F 4 "C23186" H 13700 8650 50  0001 C CNN "LCSC Part #"
 F 5 "C23186" H 13700 8650 50  0001 C CNN "LCSC part number"
-F 6 "C23186" H 13700 8650 50  0001 C CNN "LCSC"
+F 6 "C25804" H 13700 8650 50  0001 C CNN "LCSC"
 	1    13700 8650
 	1    0    0    -1
@@
 F 4 "C23186" H 13700 8900 50  0001 C CNN "LCSC Part #"
 F 5 "C23186" H 13700 8900 50  0001 C CNN "LCSC part number"
-F 6 "C23186" H 13700 8900 50  0001 C CNN "LCSC"
+F 6 "C25804" H 13700 8900 50  0001 C CNN "LCSC"
 	1    13700 8900
 	1    0    0    -1
@@
 F 4 "C23186" H 11950 7450 50  0001 C CNN "LCSC Part #"
 F 5 "C23186" H 11950 7450 50  0001 C CNN "LCSC part number"
-F 6 "C23186" H 11950 7450 50  0001 C CNN "LCSC"
+F 6 "C25804" H 11950 7450 50  0001 C CNN "LCSC"
 	1    11950 7450
 	1    0    0    -1
@@
 F 4 "C23186" H 11950 7650 50  0001 C CNN "LCSC Part #"
 F 5 "C23186" H 11950 7650 50  0001 C CNN "LCSC part number"
-F 6 "C23186" H 11950 7650 50  0001 C CNN "LCSC"
+F 6 "C25804" H 11950 7650 50  0001 C CNN "LCSC"
 	1    11950 7650
 	1    0    0    -1
