File: Hardware/E90 Kicad Files/E90.kicad_pcb (KiCad board)
At the start: 4 copper layers, 50 x 70 mm, 92 parts, among them J1 Power Connector Conn_01x02, J10 SDIN Jumper, J11 CS_SDOUT Pre Buffer Test Point, J12 SDOUT Jumper, J13 Audio Connector In Conn_01x03, J14 Conn_02x06_Odd_Even, J15 CS Passthru Jumper Conn_01x02, J17 I2S SDIN Bypass Jumper Conn_0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, J18 PMOD Passthru, J19 I2S SDOUT Bypass Conn_01x02, J2 SWD Connector Conn_02x03, J3 Power Test Point Conn_01x02, J4 BOOT0 Test Point, J6 Audio Connector Out Conn_01x03, J7 MCLK Jumper, J8 WS Jumper, J9 SCLK Jumper, U1 AMS1117-3.3, U2 CS4344_CZZ, U3 NC7SZ125P5, U4 CS5343_CZZ, U5 STM32F407VGT60

Commit message: PCB priog
Parts:
- removed C37: 180pF, Capacitor_SMD:C_0603_1608Metric
- removed J11: CS_SDOUT Pre Buffer Test Point, Connector_PinHeader_2.54mm:PinHeader_1x01_P2.54mm_Vertical
- removed J12: SDOUT Jumper, Connector_PinHeader_2.54mm:PinHeader_2x02_P2.54mm_Vertical
- removed J13: Audio Connector In Conn_01x03, Connector_PinHeader_2.54mm:PinHeader_1x03_P2.54mm_Vertical
- removed J14: Conn_02x06_Odd_Even, Connector_PinHeader_2.54mm:PinHeader_2x06_P2.54mm_Vertical
- removed J15: CS Passthru Jumper Conn_01x02, Connector_PinHeader_2.54mm:PinHeader_1x02_P2.54mm_Vertical
- removed J17: I2S SDIN Bypass Jumper Conn_01x02, Connector_PinHeader_2.54mm:PinHeader_1x02_P2.54mm_Vertical
- removed J18: PMOD Passthru, Connector_PinHeader_2.54mm:PinHeader_1x02_P2.54mm_Vertical
- removed J19: I2S SDOUT Bypass Conn_01x02, Connector_PinHeader_2.54mm:PinHeader_1x02_P2.54mm_Vertical
- added H1: MountingHole_Pad, MountingHole:MountingHole_4.3mm_M4_Pad_Via, F.Cu at (126.5, 31.0)
- added H2: MountingHole_Pad, MountingHole:MountingHole_4.3mm_M4_Pad_Via, F.Cu at (48.5, 31.0)
- added H3: MountingHole_Pad, MountingHole:MountingHole_4.3mm_M4_Pad_Via, F.Cu at (48.5, 119.0)
- added H4: MountingHole_Pad, MountingHole:MountingHole_4.3mm_M4_Pad_Via, F.Cu at (126.5, 119.0)
- added J5: Conn_01x02, Connector_PinHeader_2.54mm:PinHeader_1x02_P2.54mm_Vertical, F.Cu at (156.3, 85.3)
- added R21: 10k, Resistor_SMD:R_0603_1608Metric, F.Cu at (89.0, 116.8)
- added R22: 1k, Resistor_SMD:R_0603_1608Metric, F.Cu at (90.2, 65.7)
- added R23: 1k, Resistor_SMD:R_0603_1608Metric, F.Cu at (90.2, 64.2)
- added R24: 1k, Resistor_SMD:R_0603_1608Metric, F.Cu at (90.2, 67.2)
- added R25: 1k, Resistor_SMD:R_0603_1608Metric, F.Cu at (74.9, 78.6)
- added R26: 1k, Resistor_SMD:R_0603_1608Metric, F.Cu at (74.9, 80.1)
- added R27: 1k, Resistor_SMD:R_0603_1608Metric, F.Cu at (74.9, 81.6)
- added R28: 1k, Resistor_SMD:R_0603_1608Metric, F.Cu at (64.3, 67.6)
- added R29: 1k, Resistor_SMD:R_0603_1608Metric, F.Cu at (67.6, 67.6)
- added R30: 1k, Resistor_SMD:R_0603_1608Metric, F.Cu at (66.0, 67.5)
- added R31: 10k, Resistor_SMD:R_0603_1608Metric, F.Cu at (80.2, 102.5)
- added R32: 10k, Resistor_SMD:R_0603_1608Metric, F.Cu at (80.2, 99.3)
- added R33: 10k, Resistor_SMD:R_0603_1608Metric, F.Cu at (94.1, 110.1)
- added R34: 10k, Resistor_SMD:R_0603_1608Metric, F.Cu at (94.1, 106.7)
- added RV1: 100k, Potentiometer_THT:Potentiometer_Piher_PT-10-V10_Vertical, F.Cu at (125.7, 81.5)
- added RV2: 10k, Potentiometer_THT:Potentiometer_Bourns_PTV09A-1_Single_Vertical, F.Cu at (120.9, 50.2)
- added RV3: R_POT_US, Potentiometer_THT:Potentiometer_Bourns_PTV09A-1_Single_Vertical, F.Cu at (96.8, 49.3)
- added RV4: R_POT_US, Potentiometer_THT:Potentiometer_Bourns_PTV09A-1_Single_Vertical, F.Cu at (73.3, 49.3)
- added RV5: R_POT_US, Potentiometer_THT:Potentiometer_Bourns_PTV09A-1_Single_Vertical, F.Cu at (49.7, 49.3)
- added U6: USBLC6-2SC6, Package_TO_SOT_SMD:SOT-23-6, F.Cu at (75.7, 43.0)
- C11: value 2.7nF -> 10uF
- C26: value 100nf -> 10uF; footprint Capacitor_SMD:C_0402_1005Metric -> Capacitor_SMD:C_0603_1608Metric
- C31: value 1uF -> 10uF; footprint Capacitor_SMD:C_0603_1608Metric -> Capacitor_SMD:C_0805_2012Metric
- C6: value 3.3uF -> 10uF
- D3: value LED_Red -> B5819W; footprint LED_SMD:LED_0603_1608Metric -> Diode_SMD:D_SOD-123
- D4: value LED_Green -> LED_RGBA; footprint LED_SMD:LED_0603_1608Metric -> LED_SMD:19-237-R6GHBHC-A01-2T
- D5: value LED_Blue -> LED_RGBA; footprint LED_SMD:LED_0603_1608Metric -> LED_SMD:19-237-R6GHBHC-A01-2T
- D6: value LED_Yellow -> LED_RGBA; footprint LED_SMD:LED_0603_1608Metric -> LED_SMD:19-237-R6GHBHC-A01-2T
- J1: value Power Connector Conn_01x02 -> Conn_01x03; footprint Connector_PinHeader_2.54mm:PinHeader_1x02_P2.54mm_Vertical -> Connector_PinHeader_2.54mm:PinHeader_1x03_P2.54mm_Vertical
- J10: value SDIN Jumper -> SJ-63073E; footprint Connector_PinHeader_2.54mm:PinHeader_2x02_P2.54mm_Vertical -> Connector_Audio:CUI_SJ-63073E
- J4: value BOOT0 Test Point -> Conn_01x03; footprint Connector_PinHeader_2.54mm:PinHeader_1x01_P2.54mm_Vertical -> Connector_PinHeader_2.54mm:PinHeader_1x03_P2.54mm_Vertical
- J6: value Audio Connector Out Conn_01x03 -> Conn_01x03
- J7: value MCLK Jumper -> USB_B_Mini; footprint Connector_PinHeader_2.54mm:PinHeader_2x02_P2.54mm_Vertical -> Connector_USB:USB_Mini-B_Lumberg_2486_01_Horizontal
- J8: value WS Jumper -> Barrel_Jack_Switch; footprint Connector_PinHeader_2.54mm:PinHeader_2x02_P2.54mm_Vertical -> Connector_BarrelJack:BarrelJack_Horizontal
- J9: value SCLK Jumper -> SJ-63073E; footprint Connector_PinHeader_2.54mm:PinHeader_2x02_P2.54mm_Vertical -> Connector_Audio:CUI_SJ-63073E
- R12, R9: value 5.1K -> 10k
- R15, R16, R17, R18: value 2k2 -> 10k
- R3: value 470 -> 10k
- R5: value 10K -> 10k
- U3: value NC7SZ125P5 -> TLV2774; footprint Package_SC_70:SOT65P210X110-5N -> Package_DIP:DIP-14_W7.62mm_LongPads
- moved R14 130.0 mm to (191.9, 94.6)
- moved R10 107.2 mm to (158.7, 57.4), turned to 0 degrees
- moved C22 106.3 mm to (167.5, 93.2), turned to 0 degrees
- moved C28 87.9 mm to (169.1, 85.5), turned to 0 degrees
- moved R8 82.6 mm to (148.1, 64.1), turned to 0 degrees
- moved R9 80.3 mm to (62.0, 39.5), turned to 90 degrees
- moved R5 77.7 mm to (160.7, 76.0), turned to 0 degrees
- moved D3 76.1 mm to (86.8, 32.3)
- moved C27 74.5 mm to (156.7, 78.5)
- moved R3 72.6 mm to (62.0, 33.0), turned to 90 degrees
- moved R12 71.3 mm to (153.1, 81.4), turned to 0 degrees
- moved J3 71.0 mm to (120.8, 39.0)
- moved D4 57.3 mm to (99.4, 64.8)
- moved J2 53.1 mm to (42.5, 75.3), turned to 0 degrees
- moved R19 52.5 mm to (79.7, 112.0)
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Connections:
- C11 pad 1: GND -> Net-(C11-Pad1)
- C12 pad 2: Net-(C12-Pad2) -> CS4344_OUT
- C26 pad 1: +3V3 -> Net-(C26-Pad1)
- C26 pad 2: GND -> ANALOG_OUT
- C31 pad 1: Net-(C31-Pad1) -> +1.65V
- C31 pad 2: Net-(C31-Pad2) -> GND
- C6 pad 1: Net-(C6-Pad1) -> ANALOG_IN
- D3 pad 1: GND -> Net-(D1-Pad1)
- D3 pad 2: Net-(D3-Pad2) -> +5V
- D4 pad 1: GND -> Net-(D4-Pad1)
- D5 pad 1: GND -> Net-(D5-Pad1)
- D6 pad 1: GND -> Net-(D6-Pad1)
- J1 pad 1: VCC -> Net-(J1-Pad1)
- J1 pad 2: GND -> BOOT0
- J10 pad 1: STM32_I2S2_SDIN -> GND
- J10 pad 2: CS_SDOUT -> ANALOG_OUT
- J10 pad 3: PMOD_SDOUT -> GND
- J4 pad 1: BOOT0 -> Net-(J4-Pad1)
- J6 pad 1: Net-(C11-Pad2) -> Net-(J6-Pad1)
- J6 pad 2: Net-(C12-Pad2) -> Net-(J6-Pad2)
- J6 pad 3: GND -> Net-(J6-Pad3)
- J7 pad 1: I2S2_MCLK -> +5V
- J7 pad 2: CS_MCLK -> USB_CONN_D-
- J7 pad 3: PMOD_MCLK -> USB_CONN_D+
- J8 pad 1: I2S2_WS -> GND
- J8 pad 2: CS_WS -> VCC
- J8 pad 3: PMOD_WS -> Net-(J8-Pad3)
- J9 pad 1: I2S2_CLK -> GND
- J9 pad 2: CS_CLK -> ANALOG_IN
- J9 pad 3: PMOD_CLK -> GND
- R10 pad 2: Net-(J11-Pad1) -> STM32_I2S2_SDIN
- R11 pad 1: Net-(J13-Pad2) -> CS5343_IN
- R12 pad 2: Net-(C31-Pad1) -> Net-(J4-Pad3)
- R15 pad 2: Net-(D3-Pad2) -> Net-(R15-Pad2)
- R16 pad 1: Net-(R16-Pad1) -> Net-(R15-Pad2)
- R16 pad 2: Net-(D4-Pad2) -> Net-(C6-Pad2)
- R17 pad 1: Net-(D5-Pad2) -> +1.65V
- R17 pad 2: Net-(R17-Pad2) -> Net-(C11-Pad1)
- R18 pad 1: Net-(R18-Pad1) -> Net-(C6-Pad2)
- R18 pad 2: Net-(D6-Pad2) -> +1.65V
- R19 pad 1: GND -> ANALOG_OUT
- R19 pad 2: BOOT0 -> GND
- R20 pad 1: GND -> +3V3
- R20 pad 2: BOOT1 -> +1.65V
- R3 pad 1: Net-(C6-Pad1) -> Net-(J1-Pad1)
- R3 pad 2: Net-(C11-Pad2) -> +3V3
- R4 pad 2: Net-(C12-Pad2) -> CS4344_OUT
- R5 pad 1: GND -> Net-(J4-Pad1)
- R5 pad 2: Net-(C6-Pad1) -> +3V3
- R9 pad 1: Net-(J13-Pad1) -> GND
- R9 pad 2: Net-(C31-Pad1) -> Net-(J1-Pad3)
- U2 pad 1: CS_SDIN -> STM_I2S2_SDOUT
- U2 pad 10: Net-(C6-Pad2) -> Net-(U2-Pad10)
- U2 pad 2: CS_CLK -> I2S2_CLK
- U2 pad 3: CS_WS -> I2S2_WS
- U2 pad 4: CS_MCLK -> I2S2_MCLK
- U3 pad 1: GND -> Net-(U3-Pad1)
- U3 pad 2: Net-(J11-Pad1) -> Net-(U3-Pad1)
- U3 pad 3: GND -> Net-(R31-Pad2)
- U3 pad 4: CS_SDOUT -> +3V3
- U3 pad 5: +3V3 -> Net-(C11-Pad1)
- U4 pad 1: Net-(J11-Pad1) -> STM32_I2S2_SDIN
- U4 pad 2: CS_CLK -> I2S2_CLK
- U4 pad 3: CS_WS -> I2S2_WS
- U4 pad 4: CS_MCLK -> I2S2_MCLK
- U4 pad 8: Net-(C31-Pad2) -> Net-(U4-Pad8)
- U5 pad 17: Net-(J17-Pad1) -> STM32_I2S2_SDIN
- U5 pad 18: Net-(J19-Pad2) -> STM_I2S2_SDOUT
- U5 pad 23: Net-(U5-Pad23) -> PA0_PWM
- U5 pad 24: Net-(U5-Pad24) -> ADC1_IN1
- U5 pad 25: Net-(U5-Pad25) -> ADC1_IN2
- U5 pad 26: Net-(U5-Pad26) -> ADC1_IN3
- U5 pad 31: Net-(U5-Pad31) -> PA6_PWM
- U5 pad 32: Net-(U5-Pad32) -> PA7_PWM
- U5 pad 35: Net-(U5-Pad35) -> PB0_PWM
- U5 pad 36: Net-(U5-Pad36) -> PB1_PWM
- U5 pad 48: Net-(U5-Pad48) -> PB11_PWM
- U5 pad 59: Net-(R15-Pad1) -> PD12_PWM
- U5 pad 60: Net-(R16-Pad1) -> PD13_PWM
- U5 pad 61: Net-(R17-Pad2) -> PD14_PWM
- U5 pad 62: Net-(R18-Pad1) -> Net-(U5-Pad62)
- U5 pad 70: Net-(U5-Pad70) -> USB_D-
- U5 pad 71: Net-(U5-Pad71) -> USB_D+
- U5 pad 81: Net-(U5-Pad81) -> Net-(J6-Pad3)
- U5 pad 82: Net-(U5-Pad82) -> Net-(J6-Pad2)
- U5 pad 83: Net-(U5-Pad83) -> Net-(J6-Pad1)
Routing:
- net GND: track 92.2 -> 0.00 mm, vias 64 -> 0
- net +3V3: track 85.7 -> 0.00 mm, vias 26 -> 0
- net CS_MCLK: track 65.9 -> 0.00 mm
- net CS_WS: track 57.6 -> 0.00 mm
- net CS_CLK: track 49.6 -> 0.00 mm
- net PMOD_SDOUT: track 46.6 -> 0.00 mm
- net Net-(R18-Pad1): track 42.1 -> 0.00 mm, vias 2 -> 0
- net Net-(R17-Pad2): track 39.5 -> 0.00 mm, vias 2 -> 0
- net Net-(R16-Pad1): track 37.0 -> 0.00 mm, vias 2 -> 0
- net PMOD_SDIN: track 35.1 -> 0.00 mm
- net Net-(R15-Pad1): track 34.3 -> 0.00 mm, vias 2 -> 0
- net CS_SDOUT: track 33.0 -> 0.00 mm
- net NRST: track 32.9 -> 0.00 mm, vias 1 -> 0
- net SWO: track 30.0 -> 0.00 mm
- net CS_SDIN: track 25.5 -> 0.00 mm
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- removed copper zone on In2.Cu, net +3V3
- removed copper zone on In1.Cu, net GND
Other:
- board size 50 x 70 mm -> 90 x 100 mm
- board text removed: "+"
- board text removed: "3.3V"
- board text removed: "3.3V TP"
- board text removed: "CS PT"
- board text removed: "E90 1.0 Skyler Cornell"
- board text removed: "GND"
- board text removed: "In"
- board text removed: "L"
- board text removed: "NRST"
- board text removed: "Out"
- board text removed: "PD12"
- board text removed: "PD14"
- board text removed: "PD15"
- board text removed: "PMOD PT"
- board text removed: "Pre-Buffer TP"
- board text removed: "R"
- board text removed: "STM32 SDIN"
- board text removed: "STM32 SDOUT"
- board text removed: "SWCLK"
- board text removed: "SWD"
- board text removed: "SWDIO"
- board text removed: "SWO"
- board text removed: "VCC"

Commit message: routing
Parts:
- moved R14 122.8 mm to (69.2, 88.2), turned to 90 degrees
- moved J5 108.2 mm to (48.2, 90.0)
- moved C28 108.2 mm to (62.5, 67.0), turned to 180 degrees
- moved R5 103.7 mm to (66.5, 32.5), turned to 90 degrees
- moved C22 101.7 mm to (66.0, 87.0), turned to 270 degrees
- moved R12 96.4 mm to (66.5, 39.0), turned to 90 degrees
- moved R10 78.9 mm to (85.8, 87.5), turned to 90 degrees
- moved C27 77.1 mm to (80.0, 70.5)
- moved R8 76.1 mm to (76.5, 89.8), turned to 180 degrees
- moved J3 47.6 mm to (73.5, 33.8)
- moved R27 23.9 mm to (85.8, 60.2), turned to 180 degrees
- moved R25 22.6 mm to (85.8, 58.8), turned to 180 degrees
- moved R26 21.3 mm to (85.8, 61.8), turned to 180 degrees
- moved D2 17.4 mm to (114.0, 44.2), turned to 0 degrees
- moved D1 13.0 mm to (103.0, 27.8)
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Connections:
- R22 pad 2: Net-(D4-Pad1) -> Net-(D4-Pad2)
- R23 pad 2: Net-(D4-Pad2) -> Net-(D4-Pad3)
- R24 pad 2: Net-(D4-Pad3) -> Net-(D4-Pad1)
- R26 pad 1: PB1_PWM -> PB0_PWM
- R27 pad 1: PB0_PWM -> PB1_PWM
Routing:
- net +3V3: track 0.00 -> 91.4 mm, vias 0 -> 39
- net GND: track 0.00 -> 82.9 mm, vias 0 -> 56
- net Net-(R15-Pad1): track 0.00 -> 46.2 mm
- net CS5343_IN: track 0.00 -> 43.8 mm
- net +1.65V: track 0.00 -> 43.8 mm, vias 0 -> 2
- net STM_I2S2_SDOUT: track 0.00 -> 28.8 mm, vias 0 -> 2
- net STM32_I2S2_SDIN: track 0.00 -> 24.0 mm
- net SWDIO: track 0.00 -> 22.3 mm
- net I2S2_CLK: track 0.00 -> 21.1 mm
- net I2S2_WS: track 0.00 -> 20.6 mm
- net I2S2_MCLK: track 0.00 -> 19.8 mm
- net ANALOG_OUT: track 0.00 -> 15.6 mm
- net HSE_IN: track 0.00 -> 12.5 mm
- net VCC: track 0.00 -> 12.4 mm
- net Net-(C32-Pad2): track 0.00 -> 12.1 mm
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- added copper zone on In2.Cu, net +3V3
- added copper zone on In1.Cu, net GND

Commit message: finished pcb
Parts:
- Output Volume: renamed from RV2
- Power On: renamed from D2
- SWD Programmer: renamed from J2
- moved R9 31.5 mm to (87.1, 32.5), turned to 180 degrees
- moved J3 27.3 mm to (47.3, 41.5), turned to 180 degrees
- moved R12 22.9 mm to (86.9, 28.8), turned to 180 degrees
- moved J7 22.0 mm to (64.8, 31.5)
- moved U6 21.1 mm to (65.2, 42.2)
- moved J1 18.6 mm to (78.1, 32.5), turned to 90 degrees
- moved R3 18.1 mm to (74.4, 32.4), turned to 180 degrees
- moved J4 15.6 mm to (78.2, 28.8), turned to 90 degrees
- moved InputGain1 9.32 mm to (118.3, 87.2), turned to 0 degrees
- moved R5 8.67 mm to (74.3, 28.8), turned to 180 degrees
- moved C24 6.87 mm to (107.1, 81.5)
- moved C25 6.87 mm to (105.2, 82.5)
- moved FB4 6.87 mm to (103.9, 81.0)
- moved C23 6.87 mm to (101.8, 82.6)
- moved R7 6.87 mm to (109.0, 81.3)
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- renumbered RV5 to ADC1_IN1, RV4 to ADC1_IN2, RV3 to ADC1_IN3, RV1 to InputGain1
Connections:
- ADC1_IN1 pad 2: ADC1_IN3 -> ADC1_IN1
- ADC1_IN3 pad 2: ADC1_IN1 -> ADC1_IN3
- R25 pad 1: PB11_PWM -> PB0_PWM
- R26 pad 1: PB0_PWM -> PB11_PWM
- R28 pad 1: PD14_PWM -> PD12_PWM
- R29 pad 1: PD12_PWM -> PD14_PWM
- R29 pad 2: Net-(D6-Pad3) -> Net-(D6-Pad2)
- R30 pad 2: Net-(D6-Pad2) -> Net-(D6-Pad3)
Routing:
- net Net-(C11-Pad2): track 0.00 -> 134.8 mm, vias 0 -> 1
- net BOOT1: track 0.00 -> 59.6 mm, vias 0 -> 1
- net BOOT0: track 0.00 -> 59.2 mm, vias 0 -> 1
- net ADC1_IN3: track 0.00 -> 54.4 mm, vias 0 -> 1
- net GND: track 82.9 -> 133.0 mm, vias 56 -> 86
- net ADC1_IN1: track 0.00 -> 46.1 mm, vias 0 -> 1
- net ADC1_IN2: track 0.00 -> 38.9 mm, vias 0 -> 1
- net PA0_PWM: track 0.00 -> 38.5 mm, vias 0 -> 2
- net I2S2_MCLK: track 19.8 -> 58.2 mm
- net PD12_PWM: track 0.00 -> 34.2 mm, vias 0 -> 2
- net PD13_PWM: track 0.00 -> 33.1 mm, vias 0 -> 2
- net +5V: track 11.5 -> 44.0 mm
- net PD14_PWM: track 0.00 -> 32.1 mm, vias 0 -> 2
- net PA6_PWM: track 0.00 -> 31.0 mm, vias 0 -> 2
- net CS4344_OUT: track 2.25 -> 33.1 mm
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Other:
- board text added: "+"
- board text added: "3.3V"
- board text added: "GND"
- board text added: "I2C1"
- board text added: "Input"
- board text added: "Input Gain"
- board text added: "Output"
- board text added: "PB6"
- board text added: "PB7"
- board text added: "PD0"
- board text added: "PD1"
- board text added: "PD2"
- board text added: "SWCLK"
- board text added: "SWDIO"
- board text added: "SWO"

Commit message: added PCB image
Parts:
- added G***: LOGO, center_neg:Untitled, F.Cu at (119.4, 31.9)
- SWD: renamed from SWD Programmer
- moved D3 4.50 mm to (95.0, 30.6)
- moved C1 2.60 mm to (92.5, 39.4)
- moved C2 2.60 mm to (102.4, 38.6)
- moved D1 2.60 mm to (100.4, 27.9)
- moved FB1 2.60 mm to (96.2, 33.1)
- moved Power On 2.60 mm to (111.4, 44.4)
- moved R1 2.60 mm to (102.4, 42.1)
- moved U1 2.60 mm to (97.5, 39.6)
- moved J8 2.50 mm to (111.5, 39.2)
Routing:
- net +5V: track 44.0 -> 41.8 mm
Other:
- board text added: "+ BOOT0 -"
- board text added: "+ BOOT1 -"
- board text added: "9V"
- board text added: "GPIO"
- board text added: "I2C"
- board text added: "JLCJLCJLCJLC"
- board text added: "Skyler Cornell E90 Audio DSP REV2"
- board text added: "https://github.com/Skyler-Cornell/E90"
- board text removed: "I2C1"
