File: Hardware/E90 Kicad Files/E90.kicad_pcb (KiCad board)
At the start: 4 copper layers, 90 x 100 mm, 109 parts, among them J1 Conn_01x03, J10 SJ-63073E, J3 Power Test Point Conn_01x02, J4 Conn_01x03, J5 Conn_01x02, J6 Conn_01x03, J7 USB_B_Mini, J8 Barrel_Jack_Switch, J9 SJ-63073E, U1 AMS1117-3.3, U2 CS4344_CZZ, U3 TLV2774, U4 CS5343_CZZ, U5 STM32F407VGT60, U6 USBLC6-2SC6

Commit message: iir
Other:
- board text removed: "JLCJLCJLCJLC"
Changed lines of the file:
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@@
   (general
     (thickness 1.6)
-    (drawings 42)
+    (drawings 41)
     (tracks 1022)
     (zones 0)
@@
     )
   )
-  (gr_text JLCJLCJLCJLC (at 68.75 78.9) (layer F.SilkS)
-    (effects (font (size 1 1) (thickness 0.15)))
-  )
   (gr_circle (center 81.5 97.75) (end 81.625044 97.75) (layer F.SilkS) (width 0.3))
